Commit message: update contact dynamics

File: src/monoped_description/urdf/robot_core.xacro (robot description, xacro)
@@ -6,5 +6,5 @@
     <xacro:include filename="gazebo_full.xacro" />
     <!-- WORLD -->
-    <link name="world"/>
+    <!-- <link name="world"/>
     <joint name="world_to_body" type="prismatic">
         <origin xyz="0 0 0" rpy="0 0 0"/>
@@ -13,5 +13,5 @@
         <axis xyz="0 0 1"/>
         <limit lower="-10" upper="10" effort="1000" velocity="1000"/>
-    </joint>
+    </joint> -->
     <!-- BODY -->
     <link name="body_link">
@@ -43,12 +43,12 @@
             <origin xyz="0 0 0" rpy="0 0 0"/>
             <geometry>
-                <cylinder radius="0.05" length="0.1"/>
+                <cylinder radius="${ul_r}" length="${ul_l}"/>
             </geometry>
             <material name="yellow"/>
         </visual>
         <collision>
-            <origin xyz="0 0 0"/>
+            <origin xyz="0 0 0.025"/>
             <geometry>
-                <cylinder radius="${ul_r}" length="${ul_l}"/>
+                <cylinder radius="${ul_r}" length="${ul_l*0.1}"/>
             </geometry>
         </collision>
@@ -63,14 +63,7 @@
         <child link="lower_leg_link"/>
         <axis xyz="0 0 1"/>
-        <limit lower="0" upper="0.08" effort="1000" velocity="1000"/>
+            <limit lower="0" upper="0.08" effort="1000" velocity="1000"/>
+            <dynamics damping="0.0" friction="0.0" spring_reference="0.0" spring_stiffness="1000.0" />
     </joint>
-    <gazebo reference="upper_leg_to_lower_leg">
-        <physics>
-            <ode>
-                <spring_stiffness>10.0</spring_stiffness>
-                <spring_reference>0.0</spring_reference>
-            </ode>
-        </physics>
-    </gazebo>
     <link name="lower_leg_link">
         <visual>
@@ -96,5 +89,5 @@
                 <contact>
                     <ode>
-                        <kp>10.0</kp>
+                        <kp>100000.0</kp>
                     </ode>
                 </contact>

File: src/monoped_description/urdf/robot_material.xacro (robot description, xacro)
@@ -5,14 +5,14 @@
     </material>
     <material name="orange">
-        <color rgba="1 0.3 0.1 1"/>
+        <color rgba="1 0.3 0.1 0.8"/>
     </material>
     <material name="blue">
-        <color rgba="0.2 0.2 1 1"/>
+        <color rgba="0.2 0.2 1 0.5"/>
     </material>
     <material name="red">
-        <color rgba="1 0 0 1"/>
+        <color rgba="1 0 0 0.8"/>
     </material>
     <material name="black">
-        <color rgba="0 0 0 1"/>
+        <color rgba="0 0 0 0.8"/>
     </material>
 </robot>

Commit message: add joint stiffness property

File: src/monoped_description/urdf/robot_core.xacro (robot description, xacro)
@@ -62,8 +62,7 @@
         <parent link="upper_leg_link"/>
         <child link="lower_leg_link"/>
-        <!-- Positive prismatic motion should drive the leg downward -->
-        <axis xyz="0 0 -1"/>
-            <limit lower="0" upper="0.08" effort="1000" velocity="1000"/>
-            <dynamics damping="0.0" friction="0.0" spring_reference="0.09" spring_stiffness="1000.0" />
+        <axis xyz="0 0 1"/>
+        <limit lower="0" upper="0.08" effort="1000" velocity="1000"/>
+        <dynamics damping="0.0" friction="0.0"/>
     </joint>
     <link name="lower_leg_link">
@@ -138,3 +137,7 @@
         <material>Gazebo/Red</material>
     </gazebo>
+    <gazebo reference="upper_leg_to_lower_leg">
+        <springReference>0.0</springReference>
+        <springStiffness>1000.0</springStiffness>
+    </gazebo>
 </robot>
