Commit message: remodel, construct controller

File: src/monoped_description/urdf/gazebo_full.xacro (robot description, xacro)
@@ -11,5 +11,5 @@
       </command_interface>
       <state_interface name="position">
-        <param name="initial_value">0.5</param>
+        <param name="initial_value">2</param>
       </state_interface>
       <state_interface name="velocity"/>
@@ -17,7 +17,7 @@
     </joint>
     <joint name="upper_leg_to_lower_leg">
-      <command_interface name="effort">
-        <param name="min">-100</param>
-        <param name="max">100</param>
+      <command_interface name="position">
+        <param name="min">0.0</param>
+        <param name="max">0.09</param>
       </command_interface>
       <state_interface name="position">
@@ -33,8 +33,8 @@
     </plugin>
     <!-- Sensor Manager (จำเป็นสำหรับ IMU, Lidar, ฯลฯ) -->
-    <plugin filename="libignition-gazebo-sensors-system.so"
+    <!-- <plugin filename="libignition-gazebo-sensors-system.so"
             name="ignition::gazebo::systems::Sensors">
       <render_engine>ogre2</render_engine>
-    </plugin>
+    </plugin> -->
   </gazebo>
   <!-- Plugin mimic สำหรับทางด้านซ้าย -->

File: src/monoped_description/urdf/inertial_macros.xacro (robot description, xacro)
@@ -1,3 +1,23 @@
 <?xml version="1.0"?>
 <robot xmlns:xacro="http://www.ros.org/wiki/xacro" >
+    <!-- Specify some standard inertial calculations https://en.wikipedia.org/wiki/List_of_moments_of_inertia -->
+    <!-- These make use of xacro's mathematical functionality -->
+    <xacro:macro name="inertial_box" params="mass x y z *origin">
+        <inertial>
+            <xacro:insert_block name="origin"/>
+            <mass value="${mass}" />
+            <inertia ixx="${(1/12) * mass * (y*y+z*z)}" ixy="0.0" ixz="0.0"
+                    iyy="${(1/12) * mass * (x*x+z*z)}" iyz="0.0"
+                    izz="${(1/12) * mass * (x*x+y*y)}" />
+        </inertial>
+    </xacro:macro>
+    <xacro:macro name="inertial_cylinder" params="mass length radius *origin">
+        <inertial>
+            <xacro:insert_block name="origin"/>
+            <mass value="${mass}" />
+            <inertia ixx="${(1/12) * mass * (3*radius*radius + length*length)}" ixy="0.0" ixz="0.0"
+                    iyy="${(1/12) * mass * (3*radius*radius + length*length)}" iyz="0.0"
+                    izz="${(1/2) * mass * (radius*radius)}" />
+        </inertial>
+    </xacro:macro>
 </robot>

File: src/monoped_description/urdf/robot_core.xacro (robot description, xacro)
@@ -7,17 +7,17 @@
     <!-- WORLD -->
     <link name="world"/>
-    <!-- BODY -->
     <joint name="world_to_body" type="prismatic">
-        <origin xyz="0 0 0.3" rpy="0 0 0"/>
+        <origin xyz="0 0 0" rpy="0 0 0"/>
         <parent link="world"/>
         <child link="body_link"/>
         <axis xyz="0 0 1"/>
-        <limit lower="-0.3" upper="0.3" effort="1000" velocity="100"/>
+        <limit lower="-10" upper="10" effort="1000" velocity="1000"/>
     </joint>
+    <!-- BODY -->
     <link name="body_link">
         <visual>
             <origin xyz="0 0 0"/>
             <geometry>
-                <mesh filename="file:///$(find monoped_description)/meshes/body.stl"/>
+                <box size="${b_x} ${b_y} ${b_z}"/>
             </geometry>
             <material name="red"/>
@@ -26,15 +26,14 @@
             <origin xyz="0 0 0"/>
             <geometry>
-                <mesh filename="file:///$(find monoped_description)/meshes/body.stl"/>
+                <box size="${b_x} ${b_y} ${b_z}"/>
             </geometry>
         </collision>
-        <inertial>
-            <mass value="1.51"/>
-            <inertia ixx="1e-3" ixy="0.0" ixz="0.0" iyy="1e-3" iyz="0.0" izz="1e-3"/>
-        </inertial>
+        <xacro:inertial_box mass="${mass_body}" x="${b_x}" y="${b_y}" z="${b_z}">
+            <origin xyz="0 0 0" rpy="0 0 0"/>
+        </xacro:inertial_box>
     </link>
     <!-- UPPER LEG -->
     <joint name="body_to_upper_leg" type="fixed">
-        <origin xyz="0 0 -0.075" rpy="0 0 0"/>
+        <origin xyz="0 0 -0.125" rpy="0 0 0"/>
         <parent link="body_link"/>
         <child link="upper_leg_link"/>
@@ -42,53 +41,68 @@
     <link name="upper_leg_link">
         <visual>
-            <origin xyz="0 0 0" rpy="${pi/2} 0 0"/>
+            <origin xyz="0 0 0" rpy="0 0 0"/>
             <geometry>
-                <mesh filename="file:///$(find monoped_description)/meshes/upper_leg.stl"/>
+                <cylinder radius="0.05" length="0.1"/>
             </geometry>
-            <material name="white"/>
+            <material name="yellow"/>
         </visual>
         <collision>
-            <origin xyz="0 0 0" rpy="${pi/2} 0 0"/>
+            <origin xyz="0 0 0"/>
             <geometry>
-                <mesh filename="file:///$(find monoped_description)/meshes/upper_leg.stl"/>
+                <cylinder radius="${ul_r}" length="${ul_l}"/>
             </geometry>
         </collision>
-        <inertial>
-            <mass value="0.211"/>
-            <inertia ixx="1e-3" ixy="0.0" ixz="0.0" iyy="1e-3" iyz="0.0" izz="1e-3"/>
-        </inertial>
+        <xacro:inertial_cylinder mass="${mass_upper_leg}" radius="${ul_r}" length="${ul_l}">
+            <origin xyz="0 0 0" rpy="0 0 0"/>
+        </xacro:inertial_cylinder>
     </link>
     <!-- LOWER LEG -->
     <joint name="upper_leg_to_lower_leg" type="prismatic">
-        <origin xyz="0 0 -0.06" rpy="0 0 0"/>
+        <origin xyz="0 0 -0.1" rpy="0 0 0"/>
         <parent link="upper_leg_link"/>
         <child link="lower_leg_link"/>
         <axis xyz="0 0 1"/>
-        <limit lower="0" upper="0.05" effort="100" velocity="100"/>
-        <dynamics damping="${joint_damping}"/>
+        <limit lower="0" upper="0.08" effort="1000" velocity="1000"/>
     </joint>
+    <gazebo reference="upper_leg_to_lower_leg">
+        <physics>
+            <ode>
+                <spring_stiffness>10.0</spring_stiffness>
+                <spring_reference>0.0</spring_reference>
+            </ode>
+        </physics>
+    </gazebo>
     <link name="lower_leg_link">
         <visual>
-            <origin xyz="0 0 0" rpy="${pi/2} 0 0"/>
+            <origin xyz="0 0 0" rpy="0 0 0"/>
             <geometry>
-                <mesh filename="file:///$(find monoped_description)/meshes/lower_leg.stl"/>
+                <cylinder radius="${ll_r}" length="${ll_l}"/>
             </geometry>
             <material name="orange"/>
         </visual>
         <collision>
-            <origin xyz="0 0 0" rpy="${pi/2} 0 0"/>
+            <origin xyz="0 0 0"/>
             <geometry>
-                <mesh filename="file:///$(find monoped_description)/meshes/lower_leg.stl"/>
+                <cylinder radius="${ll_r}" length="${ll_l}"/>
             </geometry>
-            <contact_coefficients mu="0" kp="200" kd="0"/>
         </collision>
-        <inertial>
-            <mass value="0.247"/>
-            <inertia ixx="1e-3" ixy="0.0" ixz="0.0" iyy="1e-3" iyz="0.0" izz="1e-3"/>
-        </inertial>
+        <xacro:inertial_cylinder mass="${mass_lower_leg}" radius="${ll_r}" length="${ll_l}">
+            <origin xyz="0 0 0" rpy="0 0 0"/>
+        </xacro:inertial_cylinder>
     </link>
+    <gazebo reference="lower_leg_link">
+        <collision>
+            <surface>
+                <contact>
+                    <ode>
+                        <kp>10.0</kp>
+                    </ode>
+                </contact>
+            </surface>
+        </collision>
+    </gazebo>
     <!-- FOOT -->
     <joint name="lower_leg_to_foot" type="fixed">
-        <origin xyz="0 0 -0.035" rpy="0 0 0"/>
+        <origin xyz="0 0 -0.05" rpy="0 0 0"/>
         <parent link="lower_leg_link"/>
         <child link="foot_link"/>
@@ -96,20 +110,37 @@
     <link name="foot_link">
         <visual>
-            <origin xyz="0 0 0" rpy="${pi/2} 0 0"/>
+            <origin xyz="0 0 0" rpy="0 0 0"/>
             <geometry>
-                <mesh filename="file:///$(find monoped_description)/meshes/foot.stl"/>
+                <box size="${f_x} ${f_y} ${f_z}"/>
             </geometry>
             <material name="blue"/>
         </visual>
         <collision>
-            <origin xyz="0 0 0" rpy="${pi/2} 0 0"/>
+            <origin xyz="0 0 0"/>
             <geometry>
-                <mesh filename="file:///$(find monoped_description)/meshes/foot.stl"/>
+                <box size="${f_x} ${f_y} ${f_z}"/>
             </geometry>
         </collision>
-        <inertial>
-            <mass value="0.186"/>
-            <inertia ixx="1e-3" ixy="0.0" ixz="0.0" iyy="1e-3" iyz="0.0" izz="1e-3"/>
-        </inertial>
+        <xacro:inertial_box mass="${mass_foot}" x="${f_x}" y="${f_y}" z="${f_z}">
+            <origin xyz="0 0 0" rpy="0 0 0"/>
+        </xacro:inertial_box>
     </link>
+    <!-- FOOT CONTACT -->
+    <joint name="foot_to_foot_contact" type="fixed">
+        <parent link="foot_link"/>
+        <child link="foot_contact"/>
+        <origin xyz="0 0 -${f_z*0.5}"/>
+    </joint>
+    <link name="foot_contact">
+        <visual>
+            <origin xyz="0 0 0"/>
+            <geometry>
+                <sphere radius="${fc_r}"/>
+            </geometry>
+            <material name="black"/>
+        </visual>
+    </link>
+    <gazebo reference="body_link">
+        <material>Gazebo/Red</material>
+    </gazebo>
 </robot>

File: src/monoped_description/urdf/robot_material.xacro (robot description, xacro)
@@ -1,6 +1,6 @@
 <?xml version="1.0"?>
 <robot xmlns:xacro="http://www.ros.org/wiki/xacro" >
-    <material name="white">
-        <color rgba="1 1 1 1" />
+    <material name="yellow">
+        <color rgba="1 1 0 0.5"/>
     </material>
     <material name="orange">
@@ -13,3 +13,6 @@
         <color rgba="1 0 0 1"/>
     </material>
+    <material name="black">
+        <color rgba="0 0 0 1"/>
+    </material>
 </robot>

File: src/monoped_description/urdf/robot_params.xacro (robot description, xacro)
@@ -1,6 +1,29 @@
 <?xml version="1.0"?>
 <robot xmlns:xacro="http://www.ros.org/wiki/xacro" >
-    <xacro:property name="joint_damping" value="0.1"/>
-    <xacro:property name="joint_friction" value="0.05"/>
+    <!-- body/box -->
+    <xacro:property name="b_x" value="0.15"/>
+    <xacro:property name="b_y" value="0.15"/>
+    <xacro:property name="b_z" value="0.15"/>
+    <!-- upper_leg/cyclinder -->
+    <xacro:property name="ul_r" value="0.05"/>
+    <xacro:property name="ul_l" value="0.1"/>
+    <!-- lower_leg/cyclinder -->
+    <xacro:property name="ll_r" value="0.025"/>
+    <xacro:property name="ll_l" value="0.1"/>
+    <!-- foot/box -->
+    <xacro:property name="f_x" value="0.1"/>
+    <xacro:property name="f_y" value="0.1"/>
+    <xacro:property name="f_z" value="0.01"/>
+    <!-- foot/cyclinder -->
+    <xacro:property name="f_r" value="0.01"/>
+    <xacro:property name="f_l" value="0.15"/>
+    <!-- foot_contact/sphere -->
+    <xacro:property name="fc_r" value="0.001"/>
+    <xacro:property name="mass_body" value="1"/>
+    <xacro:property name="mass_upper_leg" value="0.001"/>
+    <xacro:property name="mass_lower_leg" value="0.001"/>
+    <xacro:property name="mass_foot" value="0.08"/>
+    <xacro:property name="joint_damping" value="0.001"/>
+    <xacro:property name="joint_friction" value="0.001"/>
     <xacro:property name="contact_stiffness" value="200"/>
     <xacro:property name="contact_damping" value="0.005"/>

Commit message: update

File: src/monoped_description/urdf/gazebo_full.xacro (robot description, xacro)
@@ -17,8 +17,5 @@
     </joint>
     <joint name="upper_leg_to_lower_leg">
-      <command_interface name="position">
-        <param name="min">0.0</param>
-        <param name="max">0.09</param>
-      </command_interface>
+      <command_interface name="effort"/>
       <state_interface name="position">
         <param name="initial_value">0.0</param>

File: src/monoped_description/urdf/inertial_macros.xacro (robot description, xacro)
@@ -21,3 +21,12 @@
         </inertial>
     </xacro:macro>
+    <xacro:macro name="inertial_sphere" params="mass radius *origin">
+        <inertial>
+            <xacro:insert_block name="origin"/>
+            <mass value="${mass}" />
+            <inertia ixx="${(2/5) * mass * radius * radius}" ixy="0.0" ixz="0.0"
+                    iyy="${(2/5) * mass * radius * radius}" iyz="0.0"
+                    izz="${(2/5) * mass * radius * radius}" />
+        </inertial>
+    </xacro:macro>
 </robot>

File: src/monoped_description/urdf/robot_core.xacro (robot description, xacro)
@@ -11,5 +11,5 @@
         <parent link="world"/>
         <child link="body_link"/>
-        <axis xyz="0 0 1"/>
+        <axis xyz="0 0 -1"/>
         <limit lower="-10" upper="10" effort="1000" velocity="1000"/>
     </joint> -->
@@ -62,7 +62,8 @@
         <parent link="upper_leg_link"/>
         <child link="lower_leg_link"/>
-        <axis xyz="0 0 1"/>
+        <!-- Positive prismatic motion should drive the leg downward -->
+        <axis xyz="0 0 -1"/>
             <limit lower="0" upper="0.08" effort="1000" velocity="1000"/>
-            <dynamics damping="0.0" friction="0.0" spring_reference="0.0" spring_stiffness="1000.0" />
+            <dynamics damping="0.0" friction="0.0" spring_reference="0.09" spring_stiffness="1000.0" />
     </joint>
     <link name="lower_leg_link">

Commit message: test

File: src/monoped_description/urdf/gazebo_full.xacro (robot description, xacro)
@@ -16,5 +16,5 @@
       <state_interface name="effort"/>
     </joint>
-    <joint name="upper_leg_to_lower_leg">
+    <joint name="j1">
       <command_interface name="effort"/>
       <state_interface name="position">

Commit message: edit feedback variable

File: src/monoped_description/urdf/gazebo_full.xacro (robot description, xacro)
@@ -5,15 +5,4 @@
       <plugin>gz_ros2_control/GazeboSimSystem</plugin>
     </hardware>
-    <joint name="world_to_body">
-      <command_interface name="effort">
-        <param name="min">-100</param>
-        <param name="max">100</param>
-      </command_interface>
-      <state_interface name="position">
-        <param name="initial_value">2</param>
-      </state_interface>
-      <state_interface name="velocity"/>
-      <state_interface name="effort"/>
-    </joint>
     <joint name="upper_leg_to_lower_leg">
       <command_interface name="effort"/>
@@ -30,8 +19,7 @@
     </plugin>
     <!-- Sensor Manager (จำเป็นสำหรับ IMU, Lidar, ฯลฯ) -->
-    <!-- <plugin filename="libignition-gazebo-sensors-system.so"
-            name="ignition::gazebo::systems::Sensors">
+    <plugin filename="libignition-gazebo-sensors-system.so" name="ignition::gazebo::systems::Sensors">
       <render_engine>ogre2</render_engine>
-    </plugin> -->
+    </plugin>
   </gazebo>
   <!-- Plugin mimic สำหรับทางด้านซ้าย -->
@@ -50,15 +38,49 @@
     </plugin>
   </gazebo> -->
-  <!-- <gazebo reference="base_link">
-    <sensor name="imu_sensor" type="imu">
+  <gazebo reference="body_link">
+    <!-- <sensor name="imu_sensor" type="imu">
       <always_on>true</always_on>
       <update_rate>100.0</update_rate>
       <visualize>true</visualize>
-      <topic>/imu/data</topic>
+      <topic>/imu_data</topic>
       <gz_frame_id>world</gz_frame_id>
-      <plugin filename="libignition-gazebo-imu-system.so"
-              name="ignition::gazebo::systems::Imu"/>
+      <plugin filename="libignition-gazebo-imu-system.so" name="ignition::gazebo::systems::Imu"/>
       <pose>0 0 0 0 0 0</pose>
+    </sensor> -->
+  <sensor name="altimeter_sensor" type="altimeter">
+      <always_on>true</always_on>
+      <update_rate>100.0</update_rate>
+      <visualize>true</visualize>
+      <topic>/altimeter_data</topic>
+      <pose>0 0 0 0 0 0</pose>
+      <frame_id> "world" </frame_id>
+      <plugin filename="libignition-gazebo-altimeter-system.so" name="ignition::gazebo::systems::Altimeter"/>
     </sensor>
+  </gazebo>
+  <!-- <gazebo>
+    <plugin
+      filename="libignition-gazebo-pose-publisher.so"
+      name="ignition::gazebo::systems::PosePublisher">
+      <model_name>example</model_name>  <ros>true</ros>
+      <is_static>false</is_static>
+      <update_rate>100.0</update_rate>
+      <topic>/model/example/odom</topic>
+      <link_name>body_link</link_name>
+      <publish_odom>true</publish_odom>
+      <odom_frame>odom</odom_frame>
+      <robot_base_frame>body_link</robot_base_frame>
+    </plugin>
+  </gazebo> -->
+  <!-- <gazebo>
+    <plugin name="p3d_base_controller" filename="libgazebo_ros_p3d.so">
+      <ros>
+        <namespace>/</namespace>
+        <argument>odom@nav_msgs/msg/Odometry</argument>
+        <argument>base_link_pose@geometry_msgs/msg/PoseStamped</argument>
+      </ros>
+      <update_rate>50.0</update_rate>
+      <body_name>body_link</body_name>
+      <topicName>/odom</topicName> <frameName>odom</frameName>  <ros_topic_prefix>/odom</ros_topic_prefix>
+    </plugin>
   </gazebo> -->
 </robot>

File: src/monoped_description/urdf/inertial_macros.xacro (robot description, xacro)
@@ -21,5 +21,5 @@
         </inertial>
     </xacro:macro>
-    <xacro:macro name="inertial_sphere" params="mass radius *origin">
+    <!-- <xacro:macro name="inertial_sphere" params="mass radius *origin">
         <inertial>
             <xacro:insert_block name="origin"/>
@@ -29,4 +29,4 @@
                     izz="${(2/5) * mass * radius * radius}" />
         </inertial>
-    </xacro:macro>
+    </xacro:macro> -->
 </robot>

File: src/monoped_description/urdf/robot_core.xacro (robot description, xacro)
@@ -4,5 +4,5 @@
     <xacro:include filename="robot_params.xacro"/>
     <xacro:include filename="inertial_macros.xacro"/>
-    <xacro:include filename="gazebo_full.xacro" />
+    <!-- <xacro:include filename="gazebo_full.xacro" /> -->
     <!-- WORLD -->
     <!-- <link name="world"/>
@@ -11,5 +11,5 @@
         <parent link="world"/>
         <child link="body_link"/>
-        <axis xyz="0 0 -1"/>
+        <axis xyz="0 0 1"/>
         <limit lower="-10" upper="10" effort="1000" velocity="1000"/>
     </joint> -->
@@ -35,5 +35,5 @@
     <!-- UPPER LEG -->
     <joint name="body_to_upper_leg" type="fixed">
-        <origin xyz="0 0 -0.125" rpy="0 0 0"/>
+        <origin xyz="0 0 ${b2ul}" rpy="0 0 0"/>
         <parent link="body_link"/>
         <child link="upper_leg_link"/>
@@ -59,5 +59,5 @@
     <!-- LOWER LEG -->
     <joint name="upper_leg_to_lower_leg" type="prismatic">
-        <origin xyz="0 0 -0.1" rpy="0 0 0"/>
+        <origin xyz="0 0 ${ul2ll}" rpy="0 0 0"/>
         <parent link="upper_leg_link"/>
         <child link="lower_leg_link"/>
@@ -97,5 +97,5 @@
     <!-- FOOT -->
     <joint name="lower_leg_to_foot" type="fixed">
-        <origin xyz="0 0 -0.05" rpy="0 0 0"/>
+        <origin xyz="0 0 ${ll2f}" rpy="0 0 0"/>
         <parent link="lower_leg_link"/>
         <child link="foot_link"/>
@@ -120,5 +120,5 @@
     </link>
     <!-- FOOT CONTACT -->
-    <joint name="foot_to_foot_contact" type="fixed">
+    <!-- <joint name="foot_to_foot_contact" type="fixed">
         <parent link="foot_link"/>
         <child link="foot_contact"/>
@@ -133,5 +133,5 @@
             <material name="black"/>
         </visual>
-    </link>
+    </link> -->
     <gazebo reference="body_link">
         <material>Gazebo/Red</material>

File: src/monoped_description/urdf/robot_params.xacro (robot description, xacro)
@@ -20,4 +20,11 @@
     <!-- foot_contact/sphere -->
     <xacro:property name="fc_r" value="0.001"/>
+    <!-- joint origin z asix -->
+    <!-- fix: body2upper_leg -->
+    <xacro:property name="b2ul" value="-0.125" />
+    <!-- prismatic: upper_leg2lower_leg -->
+    <xacro:property name="ul2ll" value="-0.1" />
+    <!-- fix: lower_leg2foot -->
+    <xacro:property name="ll2f" value="-0.05" />
     <xacro:property name="mass_body" value="1"/>
     <xacro:property name="mass_upper_leg" value="0.001"/>
