Commit message: add passive spring

File: src/monoped_description/urdf/gazebo_full.xacro (robot description, xacro)
@@ -7,4 +7,11 @@
     <joint name="upper_leg_to_lower_leg">
       <command_interface name="effort"/>
+      <state_interface name="position">
+        <param name="initial_value">0.0</param>
+      </state_interface>
+      <state_interface name="velocity"/>
+      <state_interface name="effort"/>
+    </joint>
+    <joint name="lower_leg_to_passive_lower_leg">
       <state_interface name="position">
         <param name="initial_value">0.0</param>
@@ -48,5 +55,5 @@
       <pose>0 0 0 0 0 0</pose>
     </sensor> -->
-  <sensor name="altimeter_sensor" type="altimeter">
+    <sensor name="altimeter_sensor" type="altimeter">
       <always_on>true</always_on>
       <update_rate>100.0</update_rate>
@@ -54,5 +61,4 @@
       <topic>/altimeter_data</topic>
       <pose>0 0 0 0 0 0</pose>
-      <frame_id> "world" </frame_id>
       <plugin filename="libignition-gazebo-altimeter-system.so" name="ignition::gazebo::systems::Altimeter"/>
     </sensor>

File: src/monoped_description/urdf/robot_core.xacro (robot description, xacro)
@@ -1,17 +1,8 @@
-<?xml version="1.0"?>
-<robot xmlns:xacro="http://www.ros.org/wiki/xacro" name="example">
+<?xml version='1.0' encoding='UTF-8'?>
+<robot xmlns:xacro="http://www.ros.org/wiki/xacro" name="monoped">
     <xacro:include filename="robot_material.xacro"/>
     <xacro:include filename="robot_params.xacro"/>
     <xacro:include filename="inertial_macros.xacro"/>
-    <!-- <xacro:include filename="gazebo_full.xacro" /> -->
-    <!-- WORLD -->
-    <!-- <link name="world"/>
-    <joint name="world_to_body" type="prismatic">
-        <origin xyz="0 0 0" rpy="0 0 0"/>
-        <parent link="world"/>
-        <child link="body_link"/>
-        <axis xyz="0 0 1"/>
-        <limit lower="-10" upper="10" effort="1000" velocity="1000"/>
-    </joint> -->
+    <xacro:include filename="gazebo_full.xacro" />
     <!-- BODY -->
     <link name="body_link">
@@ -63,5 +54,5 @@
         <child link="lower_leg_link"/>
         <axis xyz="0 0 1"/>
-        <limit lower="0" upper="0.08" effort="1000" velocity="1000"/>
+        <limit lower="0" upper="0.08" effort="200" velocity="10"/>
         <dynamics damping="0.0" friction="0.0"/>
     </joint>
@@ -84,19 +75,29 @@
         </xacro:inertial_cylinder>
     </link>
-    <gazebo reference="lower_leg_link">
-        <collision>
-            <surface>
-                <contact>
-                    <ode>
-                        <kp>100000.0</kp>
-                    </ode>
-                </contact>
-            </surface>
-        </collision>
-    </gazebo>
+    <!-- PASSSIVE LOWER LEG -->
+    <joint name="lower_leg_to_passive_lower_leg" type="prismatic">
+        <origin xyz="0 0 ${ul2ll}" rpy="0 0 0"/>
+        <parent link="lower_leg_link"/>
+        <child link="passive_lower_leg"/>
+        <axis xyz="0 0 1"/>
+        <limit lower="0" upper="0.1" effort="1000" velocity="1000"/>
+        <dynamics damping="0.0" friction="0.0"/>
+    </joint>
+    <link name="passive_lower_leg">
+        <visual>
+            <origin xyz="0 0 0" rpy="0 0 0"/>
+            <geometry>
+                <cylinder radius="${ll_r}" length="${ll_l}"/>
+            </geometry>
+            <material name="orange"/>
+        </visual>
+        <xacro:inertial_cylinder mass="${mass_lower_leg}" radius="${ll_r}" length="${ll_l}">
+            <origin xyz="0 0 0" rpy="0 0 0"/>
+        </xacro:inertial_cylinder>
+    </link>
     <!-- FOOT -->
-    <joint name="lower_leg_to_foot" type="fixed">
+    <joint name="passive_lower_leg_to_foot" type="fixed">
         <origin xyz="0 0 ${ll2f}" rpy="0 0 0"/>
-        <parent link="lower_leg_link"/>
+        <parent link="passive_lower_leg"/>
         <child link="foot_link"/>
     </joint>
@@ -134,10 +135,11 @@
         </visual>
     </link> -->
-    <gazebo reference="body_link">
-        <material>Gazebo/Red</material>
-    </gazebo>
     <gazebo reference="upper_leg_to_lower_leg">
         <springReference>0.0</springReference>
-        <springStiffness>1000.0</springStiffness>
+        <springStiffness>${joint_stiffness}</springStiffness>
+    </gazebo>
+    <gazebo reference="lower_leg_to_passive_lower_leg">
+        <springReference>0.0</springReference>
+        <springStiffness>${joint_stiffness}</springStiffness>
     </gazebo>
 </robot>

File: src/monoped_description/urdf/robot_material.xacro (robot description, xacro)
@@ -2,14 +2,14 @@
 <robot xmlns:xacro="http://www.ros.org/wiki/xacro" >
     <material name="yellow">
-        <color rgba="1 1 0 0.5"/>
+        <color rgba="1 1 0 0.8"/>
     </material>
     <material name="orange">
-        <color rgba="1 0.3 0.1 0.8"/>
+        <color rgba="1 0.3 0.1 1"/>
     </material>
     <material name="blue">
-        <color rgba="0.2 0.2 1 0.5"/>
+        <color rgba="0.2 0.2 1 1"/>
     </material>
     <material name="red">
-        <color rgba="1 0 0 0.8"/>
+        <color rgba="1 0 0 1"/>
     </material>
     <material name="black">

File: src/monoped_description/urdf/robot_params.xacro (robot description, xacro)
@@ -27,5 +27,5 @@
     <!-- fix: lower_leg2foot -->
     <xacro:property name="ll2f" value="-0.05" />
-    <xacro:property name="mass_body" value="1"/>
+    <xacro:property name="mass_body" value="1.0"/>
     <xacro:property name="mass_upper_leg" value="0.001"/>
     <xacro:property name="mass_lower_leg" value="0.001"/>
@@ -33,5 +33,4 @@
     <xacro:property name="joint_damping" value="0.001"/>
     <xacro:property name="joint_friction" value="0.001"/>
-    <xacro:property name="contact_stiffness" value="200"/>
-    <xacro:property name="contact_damping" value="0.005"/>
+    <xacro:property name="joint_stiffness" value="1000"/>
 </robot>

Commit message: complete dung dung

File: src/monoped_description/urdf/gazebo_full.xacro (robot description, xacro)
@@ -64,4 +64,17 @@
     </sensor>
   </gazebo>
+  <gazebo reference="foot_link">
+    <sensor name="contact_sensor" type="contact">
+      <always_on>true</always_on>
+      <update_rate>100.0</update_rate>
+      <visualize>true</visualize>
+      <pose>0 0 0 0 0 0</pose>
+      <plugin filename="libignition-gazebo-contact-system.so" name="ignition::gazebo::systems::Contact"/>
+      <contact>
+        <collision>foot_collision</collision>
+        <topic>/contact_data</topic>
+      </contact>
+    </sensor>
+  </gazebo>
   <!-- <gazebo>
     <plugin

File: src/monoped_description/urdf/robot_core.xacro (robot description, xacro)
@@ -110,5 +110,5 @@
             <material name="blue"/>
         </visual>
-        <collision>
+        <collision name="foot_collision">
             <origin xyz="0 0 0"/>
             <geometry>
@@ -119,4 +119,17 @@
             <origin xyz="0 0 0" rpy="0 0 0"/>
         </xacro:inertial_box>
+        <gazebo reference="foot_link">
+            <sensor name="contact_sensor" type="contact">
+            <always_on>true</always_on>
+            <update_rate>100.0</update_rate>
+            <visualize>true</visualize>
+            <pose>0 0 0 0 0 0</pose>
+            <plugin filename="libignition-gazebo-contact-system.so" name="ignition::gazebo::systems::Contact"/>
+            <contact>
+                <collision>foot_collision</collision>
+                <topic>/contact_data</topic>
+            </contact>
+            </sensor>
+        </gazebo>
     </link>
     <!-- FOOT CONTACT -->

Commit message: update

File: src/monoped_description/urdf/gazebo_full.xacro (robot description, xacro)
@@ -1,8 +1,8 @@
 <?xml version="1.0"?>
 <robot xmlns:xacro="http://www.ros.org/wiki/xacro" name="volta">
-  <ros2_control name="GazeboSimSystem" type="system">
-    <hardware>
-      <plugin>gz_ros2_control/GazeboSimSystem</plugin>
-    </hardware>
+    <ros2_control name="GazeboSystem" type="system">
+      <hardware>
+          <plugin>gz_ros2_control/GazeboSimSystem</plugin>
+      </hardware>
     <joint name="upper_leg_to_lower_leg">
       <command_interface name="effort"/>
@@ -22,12 +22,18 @@
   </ros2_control>
   <gazebo>
+      <plugin name="gz_ros2_control::GazeboSimROS2ControlPlugin" filename="libgz_ros2_control-system.so">
+          <parameters>$(find monoped_description)/config/controller_full.yaml</parameters>
+          <parameters>$(find monoped_description)/config/gaz_ros2_ctl_use_sim.yaml</parameters>
+      </plugin>
+  </gazebo>
+  <!-- <gazebo>
     <plugin filename="gz_ros2_control-system" name="gz_ros2_control::GazeboSimROS2ControlPlugin">
       <parameters>$(find monoped_description)/config/controller_full.yaml</parameters>
-    </plugin>
+    </plugin> -->
     <!-- Sensor Manager (จำเป็นสำหรับ IMU, Lidar, ฯลฯ) -->
-    <plugin filename="libignition-gazebo-sensors-system.so" name="ignition::gazebo::systems::Sensors">
+    <!-- <plugin filename="libignition-gazebo-sensors-system.so" name="ignition::gazebo::systems::Sensors">
       <render_engine>ogre2</render_engine>
     </plugin>
-  </gazebo>
+  </gazebo> -->
   <!-- Plugin mimic สำหรับทางด้านซ้าย -->
   <!-- <gazebo>
@@ -36,5 +42,5 @@
       <mimic_joint>joint11</mimic_joint>
       <multiplier>-1.0</multiplier>
-      <offset>0.0</offset>
+      <offset>0.0</offset>ros2 topic echo /contact_data
     </plugin>
     <plugin name="mimic_right" filename="libMimicJointPlugin.so">
@@ -46,5 +52,5 @@
   </gazebo> -->
   <gazebo reference="body_link">
-    <!-- <sensor name="imu_sensor" type="imu">
+    <sensor name="imu_sensor" type="imu">
       <always_on>true</always_on>
       <update_rate>100.0</update_rate>
@@ -54,5 +60,5 @@
       <plugin filename="libignition-gazebo-imu-system.so" name="ignition::gazebo::systems::Imu"/>
       <pose>0 0 0 0 0 0</pose>
-    </sensor> -->
+    </sensor>
     <sensor name="altimeter_sensor" type="altimeter">
       <always_on>true</always_on>
@@ -65,14 +71,11 @@
   </gazebo>
   <gazebo reference="foot_link">
-    <sensor name="contact_sensor" type="contact">
-      <always_on>true</always_on>
-      <update_rate>100.0</update_rate>
-      <visualize>true</visualize>
-      <pose>0 0 0 0 0 0</pose>
-      <plugin filename="libignition-gazebo-contact-system.so" name="ignition::gazebo::systems::Contact"/>
+    <sensor name="foot_contact_sensor" type="contact">
       <contact>
         <collision>foot_collision</collision>
         <topic>/contact_data</topic>
       </contact>
+      <always_on>1</always_on>
+      <update_rate>100</update_rate>
     </sensor>
   </gazebo>

File: src/monoped_description/urdf/robot_core.xacro (robot description, xacro)
@@ -92,4 +92,10 @@
             <material name="orange"/>
         </visual>
+        <collision>
+            <origin xyz="0 0 0" rpy="0 0 0"/>
+            <geometry>
+                <cylinder radius="${ll_r}" length="${ll_l}"/>
+            </geometry>
+        </collision>
         <xacro:inertial_cylinder mass="${mass_lower_leg}" radius="${ll_r}" length="${ll_l}">
             <origin xyz="0 0 0" rpy="0 0 0"/>
@@ -119,17 +125,4 @@
             <origin xyz="0 0 0" rpy="0 0 0"/>
         </xacro:inertial_box>
-        <gazebo reference="foot_link">
-            <sensor name="contact_sensor" type="contact">
-            <always_on>true</always_on>
-            <update_rate>100.0</update_rate>
-            <visualize>true</visualize>
-            <pose>0 0 0 0 0 0</pose>
-            <plugin filename="libignition-gazebo-contact-system.so" name="ignition::gazebo::systems::Contact"/>
-            <contact>
-                <collision>foot_collision</collision>
-                <topic>/contact_data</topic>
-            </contact>
-            </sensor>
-        </gazebo>
     </link>
     <!-- FOOT CONTACT -->

Commit message: update

File: src/monoped_description/urdf/gazebo_full.xacro (robot description, xacro)
@@ -27,28 +27,4 @@
       </plugin>
   </gazebo>
-  <!-- <gazebo>
-    <plugin filename="gz_ros2_control-system" name="gz_ros2_control::GazeboSimROS2ControlPlugin">
-      <parameters>$(find monoped_description)/config/controller_full.yaml</parameters>
-    </plugin> -->
-    <!-- Sensor Manager (จำเป็นสำหรับ IMU, Lidar, ฯลฯ) -->
-    <!-- <plugin filename="libignition-gazebo-sensors-system.so" name="ignition::gazebo::systems::Sensors">
-      <render_engine>ogre2</render_engine>
-    </plugin>
-  </gazebo> -->
-  <!-- Plugin mimic สำหรับทางด้านซ้าย -->
-  <!-- <gazebo>
-    <plugin name="mimic_left" filename="libMimicJointPlugin.so">
-      <master_joint>joint7</master_joint>
-      <mimic_joint>joint11</mimic_joint>
-      <multiplier>-1.0</multiplier>
-      <offset>0.0</offset>ros2 topic echo /contact_data
-    </plugin>
-    <plugin name="mimic_right" filename="libMimicJointPlugin.so">
-      <master_joint>joint8</master_joint>
-      <mimic_joint>joint12</mimic_joint>
-      <multiplier>-1.0</multiplier>
-      <offset>0.0</offset>
-    </plugin>
-  </gazebo> -->
   <gazebo reference="body_link">
     <sensor name="imu_sensor" type="imu">
@@ -70,39 +46,3 @@
     </sensor>
   </gazebo>
-  <gazebo reference="foot_link">
-    <sensor name="foot_contact_sensor" type="contact">
-      <contact>
-        <collision>foot_collision</collision>
-        <topic>/contact_data</topic>
-      </contact>
-      <always_on>1</always_on>
-      <update_rate>100</update_rate>
-    </sensor>
-  </gazebo>
-  <!-- <gazebo>
-    <plugin
-      filename="libignition-gazebo-pose-publisher.so"
-      name="ignition::gazebo::systems::PosePublisher">
-      <model_name>example</model_name>  <ros>true</ros>
-      <is_static>false</is_static>
-      <update_rate>100.0</update_rate>
-      <topic>/model/example/odom</topic>
-      <link_name>body_link</link_name>
-      <publish_odom>true</publish_odom>
-      <odom_frame>odom</odom_frame>
-      <robot_base_frame>body_link</robot_base_frame>
-    </plugin>
-  </gazebo> -->
-  <!-- <gazebo>
-    <plugin name="p3d_base_controller" filename="libgazebo_ros_p3d.so">
-      <ros>
-        <namespace>/</namespace>
-        <argument>odom@nav_msgs/msg/Odometry</argument>
-        <argument>base_link_pose@geometry_msgs/msg/PoseStamped</argument>
-      </ros>
-      <update_rate>50.0</update_rate>
-      <body_name>body_link</body_name>
-      <topicName>/odom</topicName> <frameName>odom</frameName>  <ros_topic_prefix>/odom</ros_topic_prefix>
-    </plugin>
-  </gazebo> -->
 </robot>

File: src/monoped_description/urdf/inertial_macros.xacro (robot description, xacro)
@@ -21,12 +21,3 @@
         </inertial>
     </xacro:macro>
-    <!-- <xacro:macro name="inertial_sphere" params="mass radius *origin">
-        <inertial>
-            <xacro:insert_block name="origin"/>
-            <mass value="${mass}" />
-            <inertia ixx="${(2/5) * mass * radius * radius}" ixy="0.0" ixz="0.0"
-                    iyy="${(2/5) * mass * radius * radius}" iyz="0.0"
-                    izz="${(2/5) * mass * radius * radius}" />
-        </inertial>
-    </xacro:macro> -->
 </robot>

File: src/monoped_description/urdf/robot_core.xacro (robot description, xacro)
@@ -55,5 +55,5 @@
         <axis xyz="0 0 1"/>
         <limit lower="0" upper="0.08" effort="200" velocity="10"/>
-        <dynamics damping="0.0" friction="0.0"/>
+        <dynamics damping="${joint_damping}" friction="${joint_friction}"/>
     </joint>
     <link name="lower_leg_link">
@@ -82,5 +82,5 @@
         <axis xyz="0 0 1"/>
         <limit lower="0" upper="0.1" effort="1000" velocity="1000"/>
-        <dynamics damping="0.0" friction="0.0"/>
+        <dynamics damping="${joint_damping}" friction="${joint_friction}"/>
     </joint>
     <link name="passive_lower_leg">
@@ -90,5 +90,5 @@
                 <cylinder radius="${ll_r}" length="${ll_l}"/>
             </geometry>
-            <material name="orange"/>
+            <material name="green"/>
         </visual>
         <collision>
@@ -126,19 +126,4 @@
         </xacro:inertial_box>
     </link>
-    <!-- FOOT CONTACT -->
-    <!-- <joint name="foot_to_foot_contact" type="fixed">
-        <parent link="foot_link"/>
-        <child link="foot_contact"/>
-        <origin xyz="0 0 -${f_z*0.5}"/>
-    </joint>
-    <link name="foot_contact">
-        <visual>
-            <origin xyz="0 0 0"/>
-            <geometry>
-                <sphere radius="${fc_r}"/>
-            </geometry>
-            <material name="black"/>
-        </visual>
-    </link> -->
     <gazebo reference="upper_leg_to_lower_leg">
         <springReference>0.0</springReference>

File: src/monoped_description/urdf/robot_material.xacro (robot description, xacro)
@@ -16,3 +16,12 @@
         <color rgba="0 0 0 0.8"/>
     </material>
+    <material name="grey">
+        <color rgba="0.5 0.5 0.5 1"/>
+    </material>
+    <material name="white">
+        <color rgba="1 1 1 1"/>
+    </material>
+    <material name="green">
+        <color rgba="0 1 0 1"/>
+    </material>
 </robot>

File: src/monoped_description/urdf/robot_params.xacro (robot description, xacro)
@@ -31,5 +31,5 @@
     <xacro:property name="mass_lower_leg" value="0.001"/>
     <xacro:property name="mass_foot" value="0.08"/>
-    <xacro:property name="joint_damping" value="0.001"/>
+    <xacro:property name="joint_damping" value="0.1"/>
     <xacro:property name="joint_friction" value="0.001"/>
     <xacro:property name="joint_stiffness" value="1000"/>
