Commit message: update

File: src/monoped_description/urdf/robot_params.xacro (robot description, xacro)
@@ -31,6 +31,8 @@
     <xacro:property name="mass_lower_leg" value="0.001"/>
     <xacro:property name="mass_foot" value="0.08"/>
-    <xacro:property name="joint_damping" value="0.1"/>
-    <xacro:property name="joint_friction" value="0.001"/>
+    <!-- assume no damping and friction for ideal case -->
+    <xacro:property name="joint_damping" value="0.0"/>
+    <xacro:property name="joint_friction" value="0.0"/>
+    <!-- assume set joint_stiffness for prismatic joint -->
     <xacro:property name="joint_stiffness" value="1000"/>
 </robot>

Commit message: debug 1D

File: src/monoped_description/urdf/robot_params.xacro (robot description, xacro)
@@ -30,5 +30,5 @@
     <xacro:property name="mass_upper_leg" value="0.001"/>
     <xacro:property name="mass_lower_leg" value="0.001"/>
-    <xacro:property name="mass_foot" value="0.1"/>
+    <xacro:property name="mass_foot" value="0.08"/>
     <!-- assume no damping and friction for ideal case -->
     <xacro:property name="joint_damping" value="0.0"/>
