Commit message: update

File: src/monoped_2d_description/urdf/robot_core.xacro (robot description, xacro)
@@ -45,11 +45,7 @@
             </geometry>
         </collision>
-        <inertial>
+        <xacro:inertial_cylinder mass="${mass_rw}" radius="${rw_r}" length="${rw_l}">
             <origin xyz="0 0 0" rpy="0 0 0"/>
-            <mass value="${mass_rw}"/>
-            <inertia ixx="${(1/12) * mass_rw * (3*rw_r*rw_r + rw_l*rw_l)}" ixy="0.0" ixz="0.0"
-                     iyy="${(1/12) * mass_rw * (3*rw_r*rw_r + rw_l*rw_l)}" iyz="0.0"
-                     izz="${(1/2) * mass_rw * rw_r*rw_r}"/>
-        </inertial>
+        </xacro:inertial_cylinder>
     </link>
     <joint name="body_to_rw_right" type="continuous">
@@ -75,11 +71,7 @@
             </geometry>
         </collision>
-        <inertial>
+        <xacro:inertial_cylinder mass="${mass_rw}" radius="${rw_r}" length="${rw_l}">
             <origin xyz="0 0 0" rpy="0 0 0"/>
-            <mass value="${mass_rw}"/>
-            <inertia ixx="${(1/12) * mass_rw * (3*rw_r*rw_r + rw_l*rw_l)}" ixy="0.0" ixz="0.0"
-                     iyy="${(1/12) * mass_rw * (3*rw_r*rw_r + rw_l*rw_l)}" iyz="0.0"
-                     izz="${(1/2) * mass_rw * rw_r*rw_r}"/>
-        </inertial>
+        </xacro:inertial_cylinder>
     </link>
     <joint name="body_to_thigh" type="fixed">

Commit message: Update twoD.py

File: src/monoped_2d_description/urdf/robot_core.xacro (robot description, xacro)
@@ -186,4 +186,27 @@
         </xacro:inertial_cylinder>
     </link>
+    <!-- <joint name="passive_lower_leg_to_foot" type="fixed">
+        <origin xyz="0 0 ${-shank_l}" rpy="0 0 0"/>
+        <parent link="passive_shank_link"/>
+        <child link="foot_link"/>
+    </joint>
+    <link name="foot_link">
+        <visual>
+            <origin xyz="0 0 0" rpy="0 0 0"/>
+            <geometry>
+                <box size="0.1 0.3 0.01"/>
+            </geometry>
+            <material name="blue"/>
+        </visual>
+        <collision name="foot_collision">
+            <origin xyz="0 0 0"/>
+            <geometry>
+                <box size="0.1 0.3 0.01"/>
+            </geometry>
+        </collision>
+        <xacro:inertial_box mass="${mass_foot}" x="0.1" y="0.3" z="0.01">
+            <origin xyz="0 0 0" rpy="0 0 0"/>
+        </xacro:inertial_box>
+    </link> -->
     <gazebo reference="thigh_to_shank">
         <springReference>0.0</springReference>

File: src/monoped_2d_description/urdf/robot_params.xacro (robot description, xacro)
@@ -38,15 +38,15 @@
     <!-- ============== MASS PARAMETERS ============== -->
     <!-- From TD-SLIP model: concentrated body mass with light leg -->
-    <xacro:property name="mass_body" value="3.0"/>
-    <xacro:property name="mass_thigh" value="0.05"/>
-    <xacro:property name="mass_shank" value="0.05"/>
-    <xacro:property name="mass_foot" value="0.02"/>
+    <xacro:property name="mass_body" value="0.1"/>
+    <xacro:property name="mass_thigh" value="0.001"/>
+    <xacro:property name="mass_shank" value="0.001"/>
+    <xacro:property name="mass_foot" value="0.1"/>
     <!-- ============== JOINT DYNAMICS ============== -->
     <!-- TD-SLIP with damping for Phase 2 -->
-    <xacro:property name="spring_damping" value="20.0"/>
+    <xacro:property name="spring_damping" value="0.3"/>
     <xacro:property name="spring_friction" value="0.0"/>
     <!-- ============== SPRING PARAMETERS ============== -->
     <!-- Leg spring stiffness (ks) -->
-    <xacro:property name="leg_stiffness" value="1000"/>
+    <xacro:property name="leg_stiffness" value="10000"/>
     <!-- Spring rest length (L0) is defined by link lengths -->
     <!-- L0 = thigh_l + shank_l = 0.30 m -->
@@ -55,11 +55,11 @@
     <xacro:property name="spring_lower_limit" value="0.0"/>
     <xacro:property name="spring_upper_limit" value="0.1"/>
-    <xacro:property name="spring_effort_limit" value="500"/>
-    <xacro:property name="spring_velocity_limit" value="10"/>
+    <xacro:property name="spring_effort_limit" value="1000"/>
+    <xacro:property name="spring_velocity_limit" value="1000"/>
     <!-- ============== REACTION WHEEL JOINT ============== -->
     <!-- Continuous rotation for reaction wheels -->
-    <xacro:property name="rw_damping" value="0.02"/>
-    <xacro:property name="rw_friction" value="0.0"/>
-    <xacro:property name="rw_effort_limit" value="50"/>
-    <xacro:property name="rw_velocity_limit" value="200"/>
+    <xacro:property name="rw_damping" value="0.9"/>
+    <xacro:property name="rw_friction" value="0.2"/>
+    <xacro:property name="rw_effort_limit" value="10000"/>
+    <xacro:property name="rw_velocity_limit" value="100000"/>
 </robot>
