Commit message: update

File: src/monoped_2d_description/urdf/robot_params.xacro (robot description, xacro)
@@ -26,5 +26,5 @@
     <xacro:property name="rw_r" value="0.15"/>
     <xacro:property name="rw_l" value="0.04"/>
-    <xacro:property name="mass_rw" value="1.0"/>
+    <xacro:property name="mass_rw" value="0.1"/>
     <!-- Offset from body center (Y-axis) -->
     <xacro:property name="rw_y_offset" value="${b_y/2 + rw_l/2 + 0.01}"/>
@@ -38,7 +38,7 @@
     <!-- ============== MASS PARAMETERS ============== -->
     <!-- From TD-SLIP model: concentrated body mass with light leg -->
-    <xacro:property name="mass_body" value="0.1"/>
-    <xacro:property name="mass_thigh" value="0.001"/>
-    <xacro:property name="mass_shank" value="0.001"/>
+    <xacro:property name="mass_body" value="0.5"/>
+    <xacro:property name="mass_thigh" value="0.01"/>
+    <xacro:property name="mass_shank" value="0.01"/>
     <xacro:property name="mass_foot" value="0.1"/>
     <!-- ============== JOINT DYNAMICS ============== -->
@@ -48,5 +48,5 @@
     <!-- ============== SPRING PARAMETERS ============== -->
     <!-- Leg spring stiffness (ks) -->
-    <xacro:property name="leg_stiffness" value="10000"/>
+    <xacro:property name="leg_stiffness" value="1000"/>
     <!-- Spring rest length (L0) is defined by link lengths -->
     <!-- L0 = thigh_l + shank_l = 0.30 m -->
@@ -59,6 +59,6 @@
     <!-- ============== REACTION WHEEL JOINT ============== -->
     <!-- Continuous rotation for reaction wheels -->
-    <xacro:property name="rw_damping" value="0.9"/>
-    <xacro:property name="rw_friction" value="0.2"/>
+    <xacro:property name="rw_damping" value="0.1"/>
+    <xacro:property name="rw_friction" value="0.0"/>
     <xacro:property name="rw_effort_limit" value="10000"/>
     <xacro:property name="rw_velocity_limit" value="100000"/>

Commit message: final maybe...

File: src/monoped_2d_description/urdf/robot_params.xacro (robot description, xacro)
@@ -44,5 +44,5 @@
     <!-- ============== JOINT DYNAMICS ============== -->
     <!-- TD-SLIP with damping for Phase 2 -->
-    <xacro:property name="spring_damping" value="0.3"/>
+    <xacro:property name="spring_damping" value="0.2"/>
     <xacro:property name="spring_friction" value="0.0"/>
     <!-- ============== SPRING PARAMETERS ============== -->
@@ -59,7 +59,7 @@
     <!-- ============== REACTION WHEEL JOINT ============== -->
     <!-- Continuous rotation for reaction wheels -->
-    <xacro:property name="rw_damping" value="0.1"/>
+    <xacro:property name="rw_damping" value="0.0"/>
     <xacro:property name="rw_friction" value="0.0"/>
-    <xacro:property name="rw_effort_limit" value="10000"/>
+    <xacro:property name="rw_effort_limit" value="100"/>
     <xacro:property name="rw_velocity_limit" value="100000"/>
 </robot>

Commit message: update

File: src/monoped_2d_description/urdf/robot_params.xacro (robot description, xacro)
@@ -44,5 +44,5 @@
     <!-- ============== JOINT DYNAMICS ============== -->
     <!-- TD-SLIP with damping for Phase 2 -->
-    <xacro:property name="spring_damping" value="0.2"/>
+    <xacro:property name="spring_damping" value="0.0"/>
     <xacro:property name="spring_friction" value="0.0"/>
     <!-- ============== SPRING PARAMETERS ============== -->

Commit message: add twoD_copy controller

File: src/monoped_2d_description/urdf/robot_params.xacro (robot description, xacro)
@@ -41,5 +41,5 @@
     <xacro:property name="mass_thigh" value="0.01"/>
     <xacro:property name="mass_shank" value="0.01"/>
-    <xacro:property name="mass_foot" value="0.1"/>
+    <xacro:property name="mass_foot" value="0.08"/>
     <!-- ============== JOINT DYNAMICS ============== -->
     <!-- TD-SLIP with damping for Phase 2 -->
@@ -56,10 +56,10 @@
     <xacro:property name="spring_upper_limit" value="0.1"/>
     <xacro:property name="spring_effort_limit" value="1000"/>
-    <xacro:property name="spring_velocity_limit" value="1000"/>
+    <xacro:property name="spring_velocity_limit" value="10"/>
     <!-- ============== REACTION WHEEL JOINT ============== -->
     <!-- Continuous rotation for reaction wheels -->
     <xacro:property name="rw_damping" value="0.0"/>
     <xacro:property name="rw_friction" value="0.0"/>
-    <xacro:property name="rw_effort_limit" value="100"/>
-    <xacro:property name="rw_velocity_limit" value="100000"/>
+    <xacro:property name="rw_effort_limit" value="10"/>
+    <xacro:property name="rw_velocity_limit" value="3000"/>
 </robot>

File: src/monoped_description/urdf/robot_params.xacro (robot description, xacro)
@@ -30,5 +30,5 @@
     <xacro:property name="mass_upper_leg" value="0.001"/>
     <xacro:property name="mass_lower_leg" value="0.001"/>
-    <xacro:property name="mass_foot" value="0.08"/>
+    <xacro:property name="mass_foot" value="0.1"/>
     <!-- assume no damping and friction for ideal case -->
     <xacro:property name="joint_damping" value="0.0"/>
