Commit message: update model

File: src/monoped_2d_description/urdf/gazebo_full.xacro (robot description, xacro)
@@ -1,12 +1,4 @@
 <?xml version="1.0"?>
 <robot xmlns:xacro="http://www.ros.org/wiki/xacro" name="monoped_2d">
-    <!--
-    TD-SLIP 2D Running Robot with Reaction Wheels - Gazebo Configuration
-    Control Interfaces:
-    - thigh_to_shank (prismatic): Effort control for spring compression ζ
-    - body_to_rw_left (continuous): Effort control for left reaction wheel
-    - body_to_rw_right (continuous): Effort control for right reaction wheel
-    Note: Hip joint removed - using reaction wheels for attitude control
-    -->
     <ros2_control name="GazeboSystem" type="system">
         <hardware>
@@ -22,5 +14,13 @@
             <state_interface name="effort"/>
         </joint>
-        <!-- Left Reaction Wheel: Effort control for attitude -->
+        <!-- Passive Shank Joint: No command, just state interfaces -->
+        <joint name="shank_to_passive_shank">
+            <state_interface name="position">
+                <param name="initial_value">0.0</param>
+            </state_interface>
+            <state_interface name="velocity"/>
+            <state_interface name="effort"/>
+        </joint>
+        <!-- Left Reaction Wheel: Effort (torque) control for attitude -->
         <joint name="body_to_rw_left">
             <command_interface name="effort"/>
@@ -31,5 +31,5 @@
             <state_interface name="effort"/>
         </joint>
-        <!-- Right Reaction Wheel: Effort control for attitude -->
+        <!-- Right Reaction Wheel: Effort (torque) control for attitude -->
         <joint name="body_to_rw_right">
             <command_interface name="effort"/>
@@ -68,30 +68,3 @@
         </sensor>
     </gazebo>
-    <!-- Contact sensor on foot for ground detection -->
-    <gazebo reference="foot_link">
-        <sensor name="foot_contact_sensor" type="contact">
-            <always_on>true</always_on>
-            <update_rate>100.0</update_rate>
-            <topic>/foot_contact</topic>
-            <contact>
-                <collision>foot_link_collision</collision>
-            </contact>
-            <plugin filename="libignition-gazebo-contact-system.so" name="ignition::gazebo::systems::Contact"/>
-        </sensor>
-        <!-- Foot surface properties for ground contact -->
-        <collision name="foot_collision">
-            <surface>
-                <friction>
-                    <ode>
-                        <mu>1.0</mu>
-                        <mu2>1.0</mu2>
-                    </ode>
-                </friction>
-                <bounce>
-                    <restitution_coefficient>0.0</restitution_coefficient>
-                    <threshold>0.01</threshold>
-                </bounce>
-            </surface>
-        </collision>
-    </gazebo>
 </robot>

File: src/monoped_2d_description/urdf/robot_core.xacro (robot description, xacro)
@@ -5,17 +5,4 @@
     <xacro:include filename="inertial_macros.xacro"/>
     <xacro:include filename="gazebo_full.xacro" />
-    <!--
-    TD-SLIP 2D Running Robot Model with Reaction Wheels
-    Based on: Truax et al. 2024 - Torque Driven Spring Loaded Inverted Pendulum
-    Structure:
-    body_link (main mass)
-        ├── rw_left_link (continuous joint - reaction wheel left)
-        ├── rw_right_link (continuous joint - reaction wheel right)
-        └── thigh_link (fixed - upper leg)
-            └── shank_link (prismatic joint - spring compression ζ)
-                └── foot_link (cylinder - constrains to XZ plane)
-    Note: Hip joint removed - using reaction wheels for attitude control
-    -->
-    <!-- ============== BODY ============== -->
     <link name="body_link">
         <visual>
@@ -36,11 +23,10 @@
         </xacro:inertial_box>
     </link>
-    <!-- ============== REACTION WHEELS ============== -->
-    <!-- Left Reaction Wheel (Y+ side) -->
     <joint name="body_to_rw_left" type="continuous">
-        <origin xyz="0 ${rw_y_offset} 0" rpy="${pi/2} 0 0"/>
+        <origin xyz="0 ${b_y/2 + rw_l/2 + 0.01} 0" rpy="${-pi/2} 0 0"/>
         <parent link="body_link"/>
         <child link="rw_left_link"/>
         <axis xyz="0 0 1"/>
+        <limit effort="${rw_effort_limit}" velocity="${rw_velocity_limit}"/>
         <dynamics damping="${rw_damping}" friction="${rw_friction}"/>
     </joint>
@@ -59,14 +45,18 @@
             </geometry>
         </collision>
-        <xacro:inertial_cylinder mass="${mass_rw}" radius="${rw_r}" length="${rw_l}">
+        <inertial>
             <origin xyz="0 0 0" rpy="0 0 0"/>
-        </xacro:inertial_cylinder>
+            <mass value="${mass_rw}"/>
+            <inertia ixx="${(1/12) * mass_rw * (3*rw_r*rw_r + rw_l*rw_l)}" ixy="0.0" ixz="0.0"
+                     iyy="${(1/12) * mass_rw * (3*rw_r*rw_r + rw_l*rw_l)}" iyz="0.0"
+                     izz="${(1/2) * mass_rw * rw_r*rw_r}"/>
+        </inertial>
     </link>
-    <!-- Right Reaction Wheel (Y- side) -->
     <joint name="body_to_rw_right" type="continuous">
-        <origin xyz="0 ${-rw_y_offset} 0" rpy="${pi/2} 0 0"/>
+        <origin xyz="0 ${-b_y/2 - rw_l/2 - 0.01} 0" rpy="${pi/2} 0 0"/>
         <parent link="body_link"/>
         <child link="rw_right_link"/>
         <axis xyz="0 0 1"/>
+        <limit effort="${rw_effort_limit}" velocity="${rw_velocity_limit}"/>
         <dynamics damping="${rw_damping}" friction="${rw_friction}"/>
     </joint>
@@ -85,14 +75,17 @@
             </geometry>
         </collision>
-        <xacro:inertial_cylinder mass="${mass_rw}" radius="${rw_r}" length="${rw_l}">
+        <inertial>
             <origin xyz="0 0 0" rpy="0 0 0"/>
-        </xacro:inertial_cylinder>
+            <mass value="${mass_rw}"/>
+            <inertia ixx="${(1/12) * mass_rw * (3*rw_r*rw_r + rw_l*rw_l)}" ixy="0.0" ixz="0.0"
+                     iyy="${(1/12) * mass_rw * (3*rw_r*rw_r + rw_l*rw_l)}" iyz="0.0"
+                     izz="${(1/2) * mass_rw * rw_r*rw_r}"/>
+        </inertial>
     </link>
-    <!-- ============== THIGH ============== -->
-    <!-- Upper leg segment (fixed to body) -->
     <joint name="body_to_thigh" type="fixed">
         <origin xyz="0 0 ${b2thigh}" rpy="0 0 0"/>
         <parent link="body_link"/>
         <child link="thigh_link"/>
+        <axis xyz="0 1 0"/>
     </joint>
     <link name="thigh_link">
@@ -114,6 +107,5 @@
         </xacro:inertial_cylinder>
     </link>
-    <!-- ============== SHANK (SPRING LEG) ============== -->
-    <!-- Prismatic joint for spring compression (ζ) -->
+    <!-- ACTIVE Spring Joint (effort controlled) -->
     <joint name="thigh_to_shank" type="prismatic">
         <origin xyz="0 0 ${-thigh_l}" rpy="0 0 0"/>
@@ -143,9 +135,35 @@
         </xacro:inertial_cylinder>
     </link>
-    <!-- ============== FOOT ============== -->
-    <!-- Cylinder foot - constrains motion to XZ plane (forward/backward only) -->
-    <joint name="shank_to_foot" type="fixed">
+    <!-- PASSIVE Spring Joint (Gazebo spring only, no control) -->
+    <joint name="shank_to_passive_shank" type="prismatic">
+        <origin xyz="0 0 ${-shank_l}" rpy="0 0 0"/>
+        <parent link="shank_link"/>
+        <child link="passive_shank_link"/>
+        <axis xyz="0 0 1"/>
+        <limit lower="${spring_lower_limit}" upper="${spring_upper_limit}"
+               effort="1000" velocity="1000"/>
+        <dynamics damping="${spring_damping}" friction="${spring_friction}"/>
+    </joint>
+    <link name="passive_shank_link">
+        <visual>
+            <origin xyz="0 0 ${-shank_l/2}" rpy="0 0 0"/>
+            <geometry>
+                <cylinder radius="${shank_r*0.8}" length="${shank_l}"/>
+            </geometry>
+            <material name="orange"/>
+        </visual>
+        <collision>
+            <origin xyz="0 0 ${-shank_l/2}" rpy="0 0 0"/>
+            <geometry>
+                <cylinder radius="${shank_r*0.8}" length="${shank_l}"/>
+            </geometry>
+        </collision>
+        <xacro:inertial_cylinder mass="${mass_shank}" radius="${shank_r}" length="${shank_l}">
+            <origin xyz="0 0 ${-shank_l/2}" rpy="0 0 0"/>
+        </xacro:inertial_cylinder>
+    </link>
+    <joint name="passive_shank_to_foot" type="fixed">
         <origin xyz="0 0 ${-shank_l}" rpy="${pi/2} 0 0"/>
-        <parent link="shank_link"/>
+        <parent link="passive_shank_link"/>
         <child link="foot_link"/>
     </joint>
@@ -168,9 +186,11 @@
         </xacro:inertial_cylinder>
     </link>
-    <!-- ============== SPRING PHYSICS ============== -->
-    <!-- Gazebo spring for prismatic joint -->
     <gazebo reference="thigh_to_shank">
         <springReference>0.0</springReference>
         <springStiffness>${leg_stiffness}</springStiffness>
     </gazebo>
+    <gazebo reference="shank_to_passive_shank">
+        <springReference>0.0</springReference>
+        <springStiffness>${leg_stiffness}</springStiffness>
+    </gazebo>
 </robot>

File: src/monoped_2d_description/urdf/robot_params.xacro (robot description, xacro)
@@ -22,8 +22,9 @@
     <!-- ============== REACTION WHEEL PARAMETERS ============== -->
     <!-- Reaction wheels on both sides of body for attitude control -->
-    <!-- Larger radius for more inertia, thicker for visibility -->
-    <xacro:property name="rw_r" value="0.08"/>
-    <xacro:property name="rw_l" value="0.03"/>
-    <xacro:property name="mass_rw" value="0.1"/>
+    <!-- Balance: high inertia for control authority, but not too heavy -->
+    <!-- I_wheel = 0.5 * m * r^2 = 0.5 * 1.0 * 0.15^2 ≈ 0.01125 kg.m^2 per wheel -->
+    <xacro:property name="rw_r" value="0.15"/>
+    <xacro:property name="rw_l" value="0.04"/>
+    <xacro:property name="mass_rw" value="1.0"/>
     <!-- Offset from body center (Y-axis) -->
     <xacro:property name="rw_y_offset" value="${b_y/2 + rw_l/2 + 0.01}"/>
@@ -37,5 +38,5 @@
     <!-- ============== MASS PARAMETERS ============== -->
     <!-- From TD-SLIP model: concentrated body mass with light leg -->
-    <xacro:property name="mass_body" value="1.0"/>
+    <xacro:property name="mass_body" value="3.0"/>
     <xacro:property name="mass_thigh" value="0.05"/>
     <xacro:property name="mass_shank" value="0.05"/>
@@ -43,5 +44,5 @@
     <!-- ============== JOINT DYNAMICS ============== -->
     <!-- TD-SLIP with damping for Phase 2 -->
-    <xacro:property name="spring_damping" value="0.5"/>
+    <xacro:property name="spring_damping" value="20.0"/>
     <xacro:property name="spring_friction" value="0.0"/>
     <!-- ============== SPRING PARAMETERS ============== -->
@@ -58,7 +59,7 @@
     <!-- ============== REACTION WHEEL JOINT ============== -->
     <!-- Continuous rotation for reaction wheels -->
-    <xacro:property name="rw_damping" value="0.01"/>
+    <xacro:property name="rw_damping" value="0.02"/>
     <xacro:property name="rw_friction" value="0.0"/>
-    <xacro:property name="rw_effort_limit" value="10"/>
-    <xacro:property name="rw_velocity_limit" value="100"/>
+    <xacro:property name="rw_effort_limit" value="50"/>
+    <xacro:property name="rw_velocity_limit" value="200"/>
 </robot>

Commit message: debut twoD

File: src/monoped_2d_description/urdf/gazebo_full.xacro (robot description, xacro)
@@ -8,4 +8,6 @@
         <joint name="thigh_to_shank">
             <command_interface name="effort"/>
+                <param name="min">0</param>
+                <param name="max">100</param>
             <state_interface name="position">
                 <param name="initial_value">0.0</param>
@@ -25,4 +27,6 @@
         <joint name="body_to_rw_left">
             <command_interface name="effort"/>
+                <param name="min">-3</param>
+                <param name="max">3</param>
             <state_interface name="position">
                 <param name="initial_value">0.0</param>
@@ -34,4 +38,6 @@
         <joint name="body_to_rw_right">
             <command_interface name="effort"/>
+                <param name="min">-3</param>
+                <param name="max">3</param>
             <state_interface name="position">
                 <param name="initial_value">0.0</param>

File: src/monoped_2d_description/urdf/robot_params.xacro (robot description, xacro)
@@ -22,6 +22,4 @@
     <!-- ============== REACTION WHEEL PARAMETERS ============== -->
     <!-- Reaction wheels on both sides of body for attitude control -->
-    <!-- Balance: high inertia for control authority, but not too heavy -->
-    <!-- I_wheel = 0.5 * m * r^2 = 0.5 * 1.0 * 0.15^2 ≈ 0.01125 kg.m^2 per wheel -->
     <xacro:property name="rw_r" value="0.15"/>
     <xacro:property name="rw_l" value="0.04"/>
@@ -37,9 +35,8 @@
     <xacro:property name="shank2foot" value="${-shank_l/2}"/>
     <!-- ============== MASS PARAMETERS ============== -->
-    <!-- From TD-SLIP model: concentrated body mass with light leg -->
     <xacro:property name="mass_body" value="0.5"/>
     <xacro:property name="mass_thigh" value="0.01"/>
     <xacro:property name="mass_shank" value="0.01"/>
-    <xacro:property name="mass_foot" value="0.08"/>
+    <xacro:property name="mass_foot" value="0.1"/>
     <!-- ============== JOINT DYNAMICS ============== -->
     <!-- TD-SLIP with damping for Phase 2 -->
@@ -49,11 +46,9 @@
     <!-- Leg spring stiffness (ks) -->
     <xacro:property name="leg_stiffness" value="1000"/>
-    <!-- Spring rest length (L0) is defined by link lengths -->
-    <!-- L0 = thigh_l + shank_l = 0.30 m -->
     <!-- ============== SPRING JOINT LIMITS ============== -->
     <!-- Spring compression limits (meters) -->
     <xacro:property name="spring_lower_limit" value="0.0"/>
-    <xacro:property name="spring_upper_limit" value="0.1"/>
-    <xacro:property name="spring_effort_limit" value="1000"/>
+    <xacro:property name="spring_upper_limit" value="0.13"/>
+    <xacro:property name="spring_effort_limit" value="100"/>
     <xacro:property name="spring_velocity_limit" value="10"/>
     <!-- ============== REACTION WHEEL JOINT ============== -->
@@ -61,5 +56,5 @@
     <xacro:property name="rw_damping" value="0.0"/>
     <xacro:property name="rw_friction" value="0.0"/>
-    <xacro:property name="rw_effort_limit" value="10"/>
+    <xacro:property name="rw_effort_limit" value="3"/>
     <xacro:property name="rw_velocity_limit" value="3000"/>
 </robot>
